File: oscillators/wien-bridge/wien-bridge.sch (KiCad schematic (older format))
At the start: 9 parts

Commit message: quad osc
Parts:
- C1, C2: value 10n -> 15n
- RF: value 20k -> 100k
- RG: value 10k -> 100k
- VREF: value .833 -> 2.5
Changed lines of the file:
@@
 P 4750 4350
 F 0 "RG" H 4820 4396 50  0000 L CNN
-F 1 "10k" H 4820 4305 50  0000 L CNN
+F 1 "100k" H 4820 4305 50  0000 L CNN
 F 2 "" V 4680 4350 50  0001 C CNN
 F 3 "~" H 4750 4350 50  0001 C CNN
@@
 P 5250 5100
 F 0 "RF" V 5043 5100 50  0000 C CNN
-F 1 "20k" V 5134 5100 50  0000 C CNN
+F 1 "100k" V 5134 5100 50  0000 C CNN
 F 2 "" V 5180 5100 50  0001 C CNN
 F 3 "~" H 5250 5100 50  0001 C CNN
@@
 P 6750 5200
 F 0 "C1" H 6865 5246 50  0000 L CNN
-F 1 "10n" H 6865 5155 50  0000 L CNN
+F 1 "15n" H 6865 5155 50  0000 L CNN
 F 2 "" H 6788 5050 50  0001 C CNN
 F 3 "~" H 6750 5200 50  0001 C CNN
@@
 P 5650 5750
 F 0 "C2" H 5765 5796 50  0000 L CNN
-F 1 "10n" H 5765 5705 50  0000 L CNN
+F 1 "15n" H 5765 5705 50  0000 L CNN
 F 2 "" H 5688 5600 50  0001 C CNN
 F 3 "~" H 5650 5750 50  0001 C CNN
@@
 P 6250 6400
 F 0 "VREF" H 6478 6446 50  0000 L CNN
-F 1 ".833" H 6478 6355 50  0000 L CNN
+F 1 "2.5" H 6478 6355 50  0000 L CNN
 F 2 "" H 6250 6400 50  0001 C CNN
 F 3 "~" H 6250 6400 50  0001 C CNN
